Commit message: move it stuff lowkey works just need to avoid joint collisions

File: arm_moveit_config/config/Arm_URDF_2025.ros2_control.xacro (robot description, xacro)
@@ -8,11 +8,4 @@
                 <plugin>mock_components/GenericSystem</plugin>
             </hardware>
-            <joint name="virtual_joint">
-                <command_interface name="position"/>
-                <state_interface name="position">
-                  <param name="initial_value">${initial_positions['virtual_joint']}</param>
-                </state_interface>
-                <state_interface name="velocity"/>
-            </joint>
             <joint name="joint_1">
                 <command_interface name="position"/>
@@ -57,11 +50,4 @@
                 <state_interface name="velocity"/>
             </joint>
-            <joint name="camera_joint">
-                <command_interface name="position"/>
-                <state_interface name="position">
-                  <param name="initial_value">${initial_positions['camera_joint']}</param>
-                </state_interface>
-                <state_interface name="velocity"/>
-            </joint>
             <joint name="finger_joint_1">
                 <command_interface name="position"/>
