Commit message: added dummy joint to the end effector so IK works; testing with other code and actual arm needed

File: arm_moveit_config/config/Arm_URDF_2026.ros2_control.xacro (robot description, xacro)
@@ -50,4 +50,11 @@
                 <state_interface name="velocity"/>
             </joint>
+            <joint name="dummy_ee_joint">
+                <command_interface name="position"/>
+                <state_interface name="position">
+                  <param name="initial_value">${initial_positions['dummy_ee_joint']}</param>
+                </state_interface>
+                <state_interface name="velocity"/>
+            </joint>
         </ros2_control>
     </xacro:macro>

File: simulation/urdfs/Arm_URDF_2026.urdf (robot description, URDF)
Before this commit: robot Arm_URDF_2026, 7 links, 6 joints
Links:
- added link dummy_ee, mass 0
Joints:
- added joint dummy_ee_joint: type revolute, parent gripper, child dummy_ee, origin xyz=0 0 0 rpy=0 0 0, axis 0 1 0, limit lower=0 upper=0 effort=0 velocity=0

Commit message: Revert "added dummy joint to the end effector so IK works; testing with other code and actual arm needed"
This reverts commit 15006742626e94df9c6066451b173097a1c3fb40.

File: arm_moveit_config/config/Arm_URDF_2026.ros2_control.xacro (robot description, xacro)
@@ -50,11 +50,4 @@
                 <state_interface name="velocity"/>
             </joint>
-            <joint name="dummy_ee_joint">
-                <command_interface name="position"/>
-                <state_interface name="position">
-                  <param name="initial_value">${initial_positions['dummy_ee_joint']}</param>
-                </state_interface>
-                <state_interface name="velocity"/>
-            </joint>
         </ros2_control>
     </xacro:macro>

File: simulation/urdfs/Arm_URDF_2026.urdf (robot description, URDF)
Before this commit: robot Arm_URDF_2026, 8 links, 7 joints
Links:
- removed link dummy_ee
Joints:
- removed joint dummy_ee_joint
